File: kb_pcb.kicad_sch (KiCad schematic)
At the start: 0 parts

Commit message: mx_v2
Parts:
- added A1: RaspberryPi_Pico, Module:RaspberryPi_Pico_Common_Unspecified, symbol MCU_Module:RaspberryPi_Pico
Connections:
- new net: A1.13 (GND), A1.18 (GND), A1.23 (GND), A1.28 (GND), A1.3 (GND), A1.38 (GND), A1.8 (GND)
Changed lines of the file:
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@@
 	(generator_version "9.0")
 	(paper "A4")
+	(symbol
+		(lib_id "MCU_Module:RaspberryPi_Pico")
+		(at 38.1 55.88 0)
+		(unit 1)
+		(exclude_from_sim no)
+		(in_bom yes)
+		(on_board yes)
+		(dnp no)
+		(fields_autoplaced yes)
+		(property "Reference" "A1"
+			(at 40.2433 90.17 0)
+			(effects
+				(font
+					(size 1.27 1.27)
+				)
+				(justify left)
+			)
+		)
+		(property "Value" "RaspberryPi_Pico"
+			(at 40.2433 92.71 0)
+			(effects
+				(font
+					(size 1.27 1.27)
+				)
+				(justify left)
+			)
+		)
+		(property "Footprint" "Module:RaspberryPi_Pico_Common_Unspecified"
+			(at 38.1 102.87 0)
+			(effects
+				(font
+					(size 1.27 1.27)
+				)
+				(hide yes)
+			)
+		)
+		(property "Datasheet" "https://datasheets.raspberrypi.com/pico/pico-datasheet.pdf"
+			(at 38.1 105.41 0)
+			(effects
+				(font
+					(size 1.27 1.27)
+				)
+				(hide yes)
+			)
+		)
+		(property "Description" "Versatile and inexpensive microcontroller module powered by RP2040 dual-core Arm Cortex-M0+ processor up to 133 MHz, 264kB SRAM, 2MB QSPI flash; also supports Raspberry Pi Pico 2"
+			(at 38.1 107.95 0)
+			(effects
+				(font
+					(size 1.27 1.27)
+				)
+				(hide yes)
+			)
+		)
+		(pin "29"
+		)
+		(pin "4"
+		)
+		(pin "12"
+		)
+		(pin "40"
+		)
+		(pin "18"
+		)
+		(pin "32"
+		)
+		(pin "39"
+		)
+		(pin "30"
+		)
+		(pin "20"
+		)
+		(pin "23"
+		)
+		(pin "38"
+		)
+		(pin "5"
+		)
+		(pin "15"
+		)
+		(pin "24"
+		)
+		(pin "26"
+		)
+		(pin "13"
+		)
+		(pin "34"
+		)
+		(pin "1"
+		)
+		(pin "33"
+		)
+		(pin "9"
+		)
+		(pin "22"
+		)
+		(pin "2"
+		)
+		(pin "17"
+		)
+		(pin "28"
+		)
+		(pin "21"
+		)
+		(pin "10"
+		)
+		(pin "35"
+		)
+		(pin "31"
+		)
+		(pin "14"
+		)
+		(pin "11"
+		)
+		(pin "8"
+		)
+		(pin "27"
+		)
+		(pin "37"
+		)
+		(pin "3"
+		)
+		(pin "6"
+		)
+		(pin "7"
+		)
+		(pin "16"
+		)
+		(pin "19"
+		)
+		(pin "36"
+		)
+		(pin "25"
+		)
+		(instances
+			(project ""
+				(path "/c088409a-5147-46d0-a12c-d35eea6dd7e9"
+					(reference "A1")
+					(unit 1)
+				)
+			)
+		)
+	)
 	(sheet_instances
 		(path "/"
